File: WirelessPowerRxExtensionBoard.sch (EAGLE design)
At the start: 11 parts

Commit message: Integrated MCU with Voltage Doubler and Regulator
Board still needs to be routed, verify schematic with Carrick as well.
Parts:
- CFF: device resistor:C-USC0805 -> rcl:C-USC0201
Connections:
- removed net SHDN: U$1.SHDN
- net VRECT: now also U$1.SHDN
Changed lines of the file:
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@@
 <setting verticaltext="up"/>
 </settings>
-<grid distance="0.1" unitdist="inch" unit="inch" style="lines" multiple="1" display="no" altdistance="0.001" altunitdist="inch" altunit="inch"/>
+<grid distance="0.1" unitdist="inch" unit="inch" style="lines" multiple="1" display="no" altdistance="0.01" altunitdist="inch" altunit="inch"/>
 <layers>
 <layer number="1" name="Top" color="4" fill="1" visible="no" active="no"/>
@@
 <part name="CIN" library="resistor" deviceset="C-US" device="C0805" value="10uF"/>
 <part name="COUT" library="resistor" deviceset="C-US" device="C0805" value="22uF"/>
-<part name="CFF" library="resistor" deviceset="C-US" device="C0805" value="33pF"/>
 <part name="FBT" library="resistor" deviceset="R-US_" device="M0805" value="499K"/>
 <part name="FBB" library="resistor" deviceset="R-US_" device="M0805" value="287K"/>
@@
 <part name="GND2" library="SparkFun-Aesthetics" deviceset="GND" device=""/>
 <part name="GND3" library="SparkFun-Aesthetics" deviceset="GND" device=""/>
+<part name="CFF" library="rcl" deviceset="C-US" device="C0201" value="33pF"/>
 </parts>
 <sheets>
@@
 <instance part="CIN" gate="G$1" x="116.84" y="50.8"/>
 <instance part="COUT" gate="G$1" x="55.88" y="30.48"/>
-<instance part="CFF" gate="G$1" x="33.02" y="35.56"/>
 <instance part="FBT" gate="G$1" x="45.72" y="33.02" rot="R90"/>
 <instance part="FBB" gate="G$1" x="45.72" y="12.7" rot="R90"/>
@@
 <instance part="GND2" gate="1" x="50.8" y="-5.08"/>
 <instance part="GND3" gate="1" x="116.84" y="33.02"/>
+<instance part="CFF" gate="G$1" x="33.02" y="35.56"/>
 </instances>
 <busses>
@@
 <wire x1="99.06" y1="55.88" x2="116.84" y2="55.88" width="0.1524" layer="91"/>
 <wire x1="116.84" y1="55.88" x2="116.84" y2="53.34" width="0.1524" layer="91"/>
+</segment>
+<segment>
+<pinref part="U$1" gate="G$1" pin="SHDN"/>
+<wire x1="63.5" y1="55.88" x2="55.88" y2="55.88" width="0.1524" layer="91"/>
+<label x="63.246" y="57.912" size="1.778" layer="95" rot="R180"/>
 </segment>
 </net>
@@
 <pinref part="COUT" gate="G$1" pin="1"/>
 <wire x1="55.88" y1="33.02" x2="55.88" y2="40.64" width="0.1524" layer="91"/>
+<pinref part="FBT" gate="G$1" pin="2"/>
+<wire x1="45.72" y1="40.64" x2="45.72" y2="38.1" width="0.1524" layer="91"/>
+<wire x1="45.72" y1="40.64" x2="55.88" y2="40.64" width="0.1524" layer="91"/>
+<junction x="55.88" y="40.64"/>
 <pinref part="CFF" gate="G$1" pin="1"/>
 <wire x1="33.02" y1="38.1" x2="33.02" y2="40.64" width="0.1524" layer="91"/>
 <wire x1="33.02" y1="40.64" x2="45.72" y2="40.64" width="0.1524" layer="91"/>
-<pinref part="FBT" gate="G$1" pin="2"/>
-<wire x1="45.72" y1="40.64" x2="45.72" y2="38.1" width="0.1524" layer="91"/>
-<wire x1="45.72" y1="40.64" x2="55.88" y2="40.64" width="0.1524" layer="91"/>
 <junction x="45.72" y="40.64"/>
-<junction x="55.88" y="40.64"/>
 </segment>
 </net>
@@
 <pinref part="FBT" gate="G$1" pin="1"/>
 <wire x1="45.72" y1="17.78" x2="45.72" y2="22.86" width="0.1524" layer="91"/>
-<pinref part="CFF" gate="G$1" pin="2"/>
 <wire x1="45.72" y1="22.86" x2="45.72" y2="27.94" width="0.1524" layer="91"/>
 <wire x1="33.02" y1="30.48" x2="33.02" y2="22.86" width="0.1524" layer="91"/>
@@
 <junction x="45.72" y="22.86"/>
 <label x="38.1" y="22.86" size="1.778" layer="95"/>
-</segment>
-</net>
-<net name="SHDN" class="0">
-<segment>
-<pinref part="U$1" gate="G$1" pin="SHDN"/>
-<wire x1="63.5" y1="55.88" x2="55.88" y2="55.88" width="0.1524" layer="91"/>
-<label x="63.246" y="57.912" size="1.778" layer="95" rot="R180"/>
-</segment>
-</net>
+<pinref part="CFF" gate="G$1" pin="2"/>
+</segment>
+</net>
