File: WirelessPowerRxExtensionBoard/WirelessPowerRxExtensionBoard.sch (EAGLE design)
At the start: 11 parts

Commit message: Integrated MCU with Voltage Doubler and Regulator
Board still needs to be routed, verify schematic with Carrick as well.
Parts:
- added ATMEGA_3.3: ATMEGA1284PA-AU, kwgilpin:ATMEGA164PA-AU
- added B2: SWITCH-MOMENTARY, 000_carrick:SWITCH-MOMENTARY
- added C18, C19, C20, C21: 0.1uF, carrick:CAP0603
- added D5: LED red, 000_carrick:LED
- added D6: LED green, 000_carrick:LED
- added ISP: DF3-6, hirose:DF3-6
- added PWM: DF3-5, hirose:DF3-5
- added Q1, Q2, Q3: MOSFET-N, carrick:MOSFET-N
- added R17, R18, R19: 100k, carrick:RES0603
- added R23: 300, 000_carrick:RES0603
- added R24: 261, 000_carrick:RES0603
- added R26: 1k, 000_carrick:RES0603
- added U$2: INDUCTOR, crawford:INDUCTOR
- added UART0: DF3-4, hirose:DF3-4
- added XBEE: XBEE-1SML-HOLES, carrick:XBEE-1SML-HOLES
- C1, C2: value (none) -> 9F
- CFF: device resistor:C-USC0805 -> rcl:C-USC0201
- CIN, COUT: device resistor:C-USC0805 -> rcl:C-USC0805
Connections:
- removed net VOUT: CFF.1, COUT.1, FBT.2, U$1.VOUT
- new net 3.3V: ATMEGA_3.3.AREF, ATMEGA_3.3.AVCC, ATMEGA_3.3.VCC@1, ATMEGA_3.3.VCC@2, ATMEGA_3.3.VCC@3, C18.P$2, C19.P$2, C20.P$2, C21.P$2, D5.P$2, D6.P$2, ISP.P6, PWM.P4, UART0.P4, XBEE.VDD
- new net AT3_!RESET!: ATMEGA_3.3.!RESET!, ISP.P2
- new net AT3_BUTTON: ATMEGA_3.3.PD7/PCINT31/OC2A, R26.1
- new net AT3_LED1: ATMEGA_3.3.PB4/!SS!/OC0B/PCINT12, R23.2
- new net AT3_LED2: ATMEGA_3.3.PB3/AINT1/OC0A/PCINT11, R24.2
- new net AT3_PR_MISO: ATMEGA_3.3.PB6/PCINT14/MISO, ISP.P4
- new net AT3_PR_MOSI: ATMEGA_3.3.PB5/PCINT13/MOSI, ISP.P3
- new net AT3_PR_SCK: ATMEGA_3.3.PB7/PCINT15/SCK, ISP.P5
- new net AT3_RX0: ATMEGA_3.3.PD0/PCINT24/RXD0, UART0.P2
- new net AT3_RX1: ATMEGA_3.3.PD2/PCINT25/RXD1/INT0, XBEE.DOUT
- new net AT3_TX0: ATMEGA_3.3.PD1/PCINT24/TXD0, UART0.P3
- new net AT3_TX1: ATMEGA_3.3.PD3/PCINT24/TXD1/INT1, XBEE.DIN
- new net N$20: PWM.P3, Q3.D
- new net N$22: PWM.P2, Q2.D
- new net N$23: B2.P$1, R26.2
- new net N$24: PWM.P1, Q1.D
- new net N$38: D5.P$1, R23.1
- new net N$39: D6.P$1, R24.1
- new net PWM1: ATMEGA_3.3.PD4/PCINT24/XCK1/OC1B, Q1.G, R19.1
- new net PWM2: ATMEGA_3.3.PD5/PCINT29/OC1A, Q2.G, R18.1
- new net PWM3: ATMEGA_3.3.PD6/PCINT30/OC2B/ICP, Q3.G, R17.1
- new net VDOUBLE: C1.+, CIN.1, D1.C, U$1.SHDN, U$1.VIN, U$2.1
- net GND: now also ATMEGA_3.3.GND@1, ATMEGA_3.3.GND@2, ATMEGA_3.3.GND@3, ATMEGA_3.3.GND@4, B2.P$2, C18.P$1, C19.P$1, C20.P$1, C21.P$1, ISP.P1, Q1.S, Q2.S, Q3.S, R17.2, R18.2, R19.2, UART0.P1, XBEE.GND
- net SW: now also U$2.2
- net VRECT: now also CFF.1, COUT.1, FBT.2, PWM.P5, U$1.VOUT; no longer C1.+, CIN.1, D1.C, U$1.SHDN, U$1.VIN
Other:
- note added: "2011v1"
- note added: "AVcc Cap"
- note added: "Add Voltage Divider to Measure Vrect"
- note added: "Author: Carrick Detweiler <carrick@cse.unl.edu>"
- note added: "If you have room add a connector"
- note added: "Mosfets to control power to external devices"
- note added: "One Cap per Vcc pin"
- note added: "You can probably fit the processor under the radio"
- note added: "with a few general I/O pins"

Commit message: Finished Schematic for Wireless Power Rx Extension Board
Also updated crawford library to include zener diode
Parts:
- added R1, R2: 47K, resistor:R-US_M0805
- added Z1, Z2: ZENERDIODE, crawford:ZENERDIODE
- C1, C2: value 9F -> 1.5F; device resistor:CPOL-USE5-13 -> resistor:CPOL-USE5-10.5
Connections:
- removed net N$2: C1.-, C2.+, H1.P1
- removed net VRECT: CFF.1, COUT.1, FBT.2, PWM.P5, U$1.VOUT
- new net N$3: ATMEGA_3.3.PA0/ADC0/PCINT0, R1.1, R2.2
- new net N$4: C1.-, C2.+, H1.P1, Z1.A, Z2.C
- net 3.3V: now also CFF.1, COUT.1, FBT.2, U$1.VOUT
- net GND: now also R2.1, Z2.A
- net VDOUBLE: now also PWM.P5, R1.2, Z1.C
Other:
- note removed: "Add Voltage Divider to Measure Vrect"
- moved on the sheet: U$2

Commit message: First Routing Revision Complete
Much improved since the first routing!
Parts:
- R1: value 47K -> 47k; device resistor:R-US_M0805 -> carrick:RES0603
- R2: device resistor:R-US_M0805 -> carrick:RES0603
Other:
- moved on the sheet: R1, R2
Changed lines of the file:
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@@
 <setting verticaltext="up"/>
 </settings>
-<grid distance="0.01" unitdist="inch" unit="inch" style="lines" multiple="1" display="no" altdistance="0.01" altunitdist="inch" altunit="inch"/>
+<grid distance="0.1" unitdist="inch" unit="inch" style="lines" multiple="1" display="no" altdistance="0.01" altunitdist="inch" altunit="inch"/>
 <layers>
 <layer number="1" name="Top" color="4" fill="1" visible="no" active="no"/>
@@
 <layer number="95" name="Names" color="7" fill="1" visible="yes" active="yes"/>
 <layer number="96" name="Values" color="7" fill="1" visible="yes" active="yes"/>
-<layer number="97" name="Info" color="7" fill="1" visible="yes" active="yes"/>
-<layer number="98" name="Guide" color="6" fill="1" visible="yes" active="yes"/>
+<layer number="97" name="Info" color="7" fill="1" visible="no" active="yes"/>
+<layer number="98" name="Guide" color="6" fill="1" visible="no" active="yes"/>
 <layer number="100" name="Muster" color="7" fill="1" visible="no" active="no"/>
-<layer number="101" name="Patch_Top" color="12" fill="4" visible="yes" active="yes"/>
-<layer number="102" name="Vscore" color="7" fill="1" visible="yes" active="yes"/>
-<layer number="103" name="tMap" color="7" fill="1" visible="yes" active="yes"/>
-<layer number="104" name="Name" color="7" fill="1" visible="yes" active="yes"/>
-<layer number="105" name="PLATING" color="10" fill="7" visible="yes" active="yes"/>
-<layer number="106" name="BGA-Top" color="4" fill="1" visible="yes" active="yes"/>
-<layer number="107" name="BD-Top" color="5" fill="1" visible="yes" active="yes"/>
-<layer number="116" name="Patch_BOT" color="9" fill="4" visible="yes" active="yes"/>
-<layer number="121" name="_tsilk" color="7" fill="1" visible="yes" active="yes"/>
-<layer number="122" name="_bsilk" color="7" fill="1" visible="yes" active="yes"/>
+<layer number="101" name="Patch_Top" color="12" fill="4" visible="no" active="yes"/>
+<layer number="102" name="Vscore" color="7" fill="1" visible="no" active="yes"/>
+<layer number="103" name="tMap" color="7" fill="1" visible="no" active="yes"/>
+<layer number="104" name="Name" color="7" fill="1" visible="no" active="yes"/>
+<layer number="105" name="PLATING" color="10" fill="7" visible="no" active="yes"/>
+<layer number="106" name="BGA-Top" color="4" fill="1" visible="no" active="yes"/>
+<layer number="107" name="BD-Top" color="5" fill="1" visible="no" active="yes"/>
+<layer number="116" name="Patch_BOT" color="9" fill="4" visible="no" active="yes"/>
+<layer number="121" name="_tsilk" color="7" fill="1" visible="no" active="yes"/>
+<layer number="122" name="_bsilk" color="7" fill="1" visible="no" active="yes"/>
 <layer number="125" name="_tNames" color="7" fill="1" visible="no" active="yes"/>
 <layer number="144" name="Drill_legend" color="7" fill="1" visible="no" active="yes"/>
-<layer number="151" name="HeatSink" color="7" fill="1" visible="yes" active="yes"/>
+<layer number="151" name="HeatSink" color="7" fill="1" visible="no" active="yes"/>
 <layer number="200" name="200bmp" color="1" fill="10" visible="no" active="no"/>
 <layer number="201" name="201bmp" color="2" fill="1" visible="no" active="no"/>
 <layer number="202" name="202bmp" color="3" fill="1" visible="no" active="no"/>
-<layer number="203" name="203bmp" color="4" fill="10" visible="yes" active="yes"/>
-<layer number="204" name="204bmp" color="5" fill="10" visible="yes" active="yes"/>
-<layer number="205" name="205bmp" color="6" fill="10" visible="yes" active="yes"/>
-<layer number="206" name="206bmp" color="7" fill="10" visible="yes" active="yes"/>
-<layer number="207" name="207bmp" color="8" fill="10" visible="yes" active="yes"/>
-<layer number="208" name="208bmp" color="9" fill="10" visible="yes" active="yes"/>
+<layer number="203" name="203bmp" color="4" fill="10" visible="no" active="yes"/>
+<layer number="204" name="204bmp" color="5" fill="10" visible="no" active="yes"/>
+<layer number="205" name="205bmp" color="6" fill="10" visible="no" active="yes"/>
+<layer number="206" name="206bmp" color="7" fill="10" visible="no" active="yes"/>
+<layer number="207" name="207bmp" color="8" fill="10" visible="no" active="yes"/>
+<layer number="208" name="208bmp" color="9" fill="10" visible="no" active="yes"/>
 <layer number="209" name="209bmp" color="7" fill="1" visible="no" active="yes"/>
 <layer number="210" name="210bmp" color="7" fill="1" visible="no" active="yes"/>
@@
 <layer number="250" name="Descript" color="3" fill="1" visible="no" active="no"/>
 <layer number="251" name="SMDround" color="12" fill="11" visible="no" active="no"/>
-<layer number="254" name="cooling" color="7" fill="1" visible="yes" active="yes"/>
+<layer number="254" name="cooling" color="7" fill="1" visible="no" active="yes"/>
 </layers>
 <schematic xreflabel="%F%N/%S.%C%R" xrefpart="/%S.%C%R">
@@
 <part name="U$1" library="crawford" deviceset="STEPUPCONVERTER" device=""/>
 <part name="U$2" library="crawford" deviceset="INDUCTOR" device=""/>
-<part name="R2" library="resistor" deviceset="R-US_" device="M0805" value="47K"/>
-<part name="R1" library="resistor" deviceset="R-US_" device="M0805" value="47K"/>
 <part name="SUPPLY4" library="000_carrick" deviceset="GND" device=""/>
 <part name="C1" library="resistor" deviceset="CPOL-US" device="E5-10.5" value="1.5F"/>
@@
 <part name="Z1" library="crawford" deviceset="ZENERDIODE" device=""/>
 <part name="Z2" library="crawford" deviceset="ZENERDIODE" device=""/>
+<part name="R1" library="carrick" deviceset="RES" device="0603" value="47k"/>
+<part name="R2" library="carrick" deviceset="RES" device="0603" value="47K"/>
 </parts>
 <sheets>
@@
 <instance part="U$1" gate="G$1" x="93.98" y="165.1"/>
 <instance part="U$2" gate="G$1" x="99.06" y="142.24" rot="R90"/>
-<instance part="R2" gate="G$1" x="29.21" y="80.01" rot="R90"/>
-<instance part="R1" gate="G$1" x="29.21" y="92.71" rot="R90"/>
-<instance part="SUPPLY4" gate="GND" x="29.21" y="69.85"/>
+<instance part="SUPPLY4" gate="GND" x="30.48" y="71.12"/>
 <instance part="C1" gate="G$1" x="22.86" y="33.02"/>
 <instance part="C2" gate="G$1" x="22.86" y="17.78"/>
@@
 <attribute name="NAME" x="37.3634" y="13.716" size="1.778" layer="95" rot="R90"/>
 </instance>
+<instance part="R1" gate="G$1" x="27.94" y="96.52" rot="R90"/>
+<instance part="R2" gate="G$1" x="27.94" y="83.82" rot="R90"/>
 </instances>
 <busses>
@@
 </segment>
 <segment>
+<pinref part="SUPPLY4" gate="GND" pin="GND"/>
 <pinref part="R2" gate="G$1" pin="1"/>
-<wire x1="29.21" y1="74.93" x2="29.21" y2="72.39" width="0.1524" layer="91"/>
-<pinref part="SUPPLY4" gate="GND" pin="GND"/>
+<wire x1="27.94" y1="78.74" x2="30.48" y2="78.74" width="0.1524" layer="91"/>
+<wire x1="30.48" y1="78.74" x2="30.48" y2="73.66" width="0.1524" layer="91"/>
 </segment>
 </net>
@@
 <segment>
 <pinref part="R1" gate="G$1" pin="2"/>
-<wire x1="29.21" y1="97.79" x2="16.51" y2="97.79" width="0.1524" layer="91"/>
-<label x="17.78" y="99.06" size="1.778" layer="95"/>
+<wire x1="27.94" y1="101.6" x2="7.62" y2="101.6" width="0.1524" layer="91"/>
+<wire x1="7.62" y1="101.6" x2="7.62" y2="99.06" width="0.1524" layer="91"/>
+<label x="12.7" y="101.6" size="1.778" layer="95"/>
 </segment>
 </net>
@@
 <pinref part="CFF" gate="G$1" pin="2"/>
 <label x="43.18" y="139.7" size="1.778" layer="95"/>
-</segment>
-</net>
-<net name="N$3" class="0">
-<segment>
-<pinref part="ATMEGA_3.3" gate="G$1" pin="PA0/ADC0/PCINT0"/>
-<wire x1="29.21" y1="86.36" x2="45.72" y2="86.36" width="0.1524" layer="91"/>
-<pinref part="R2" gate="G$1" pin="2"/>
-<pinref part="R1" gate="G$1" pin="1"/>
-<wire x1="29.21" y1="87.63" x2="29.21" y2="86.36" width="0.1524" layer="91"/>
-<wire x1="29.21" y1="86.36" x2="29.21" y2="85.09" width="0.1524" layer="91"/>
-<junction x="29.21" y="86.36"/>
 </segment>
 </net>
@@
 </segment>
 </net>
+<net name="N$3" class="0">
+<segment>
+<pinref part="R1" gate="G$1" pin="1"/>
+<pinref part="R2" gate="G$1" pin="2"/>
+<wire x1="27.94" y1="91.44" x2="27.94" y2="88.9" width="0.1524" layer="91"/>
+<pinref part="ATMEGA_3.3" gate="G$1" pin="PA0/ADC0/PCINT0"/>
+<wire x1="45.72" y1="86.36" x2="35.56" y2="86.36" width="0.1524" layer="91"/>
+<wire x1="35.56" y1="86.36" x2="35.56" y2="88.9" width="0.1524" layer="91"/>
+<wire x1="35.56" y1="88.9" x2="27.94" y2="88.9" width="0.1524" layer="91"/>
+<junction x="27.94" y="88.9"/>
+</segment>
+</net>
